Commit message: added back the old urdf and an example of new urdf that does not work. We are going to debug it.

File: urdf/panda.urdf (robot description, URDF)
Before this commit: robot panda, 14 links, 13 joints
Links:
- removed link ball_link
- added link panda_ball
- added link panda_hand_sc; collision cylinder length=0.1 radius=0.05; collision cylinder length=0.1 radius=0.07
- added link panda_link0_sc; collision cylinder length=0.03 radius=0.09; collision sphere radius=0.09
- added link panda_link1_sc; collision cylinder length=0.283 radius=0.09; collision sphere radius=0.09
- added link panda_link2_sc; collision cylinder length=0.12 radius=0.09; collision sphere radius=0.09
- added link panda_link3_sc; collision cylinder length=0.15 radius=0.09; collision sphere radius=0.09
- added link panda_link4_sc; collision cylinder length=0.12 radius=0.09; collision sphere radius=0.09
- added link panda_link5_sc; collision cylinder length=0.1 radius=0.09; collision cylinder length=0.14 radius=0.055
- added link panda_link6_sc; collision cylinder length=0.08 radius=0.08; collision sphere radius=0.08
- added link panda_link7_sc; collision cylinder length=0.01 radius=0.06; collision cylinder length=0.14 radius=0.07
- link panda_hand: geometry collision mesh filename=package://franka_description/meshes/collision/hand.stl; visual mesh filename=package://franka_description/meshes/visual/hand.dae
- link panda_leftfinger: geometry collision box size=17.5e-3 15.2e-3 18.5e-3; collision box size=17.5e-3 7e-3 23.5e-3
- link panda_link0: geometry collision mesh filename=package://franka_description/meshes/collision/link0.stl; visual mesh filename=package://franka_description/meshes/visual/link0.dae
- link panda_link1: geometry collision mesh filename=package://franka_description/meshes/collision/link1.stl; visual mesh filename=package://franka_description/meshes/visual/link1.dae
- link panda_link2: geometry collision mesh filename=package://franka_description/meshes/collision/link2.stl; visual mesh filename=package://franka_description/meshes/visual/link2.dae
- link panda_link3: geometry collision mesh filename=package://franka_description/meshes/collision/link3.stl; visual mesh filename=package://franka_description/meshes/visual/link3.dae
- link panda_link4: geometry collision mesh filename=package://franka_description/meshes/collision/link4.stl; visual mesh filename=package://franka_description/meshes/visual/link4.dae
- link panda_link5: geometry collision mesh filename=package://franka_description/meshes/collision/link5.stl; visual mesh filename=package://franka_description/meshes/visual/link5.dae
- link panda_link6: geometry collision mesh filename=package://franka_description/meshes/collision/link6.stl; visual mesh filename=package://franka_description/meshes/visual/link6.dae
- link panda_link7: geometry collision mesh filename=package://franka_description/meshes/collision/link7.stl; visual mesh filename=package://franka_description/meshes/visual/link7.dae
- link panda_rightfinger: geometry collision box size=17.5e-3 15.2e-3 18.5e-3; collision box size=17.5e-3 7e-3 23.5e-3
Joints:
- removed joint ball_joint
- added joint panda_hand_sc_joint: type fixed, parent panda_hand, child panda_hand_sc, origin rpy=0 0 0
- added joint panda_link0_sc_joint: type fixed, parent panda_link0, child panda_link0_sc, origin rpy=0 0 0
- added joint panda_link1_sc_joint: type fixed, parent panda_link1, child panda_link1_sc, origin rpy=0 0 0
- added joint panda_link2_sc_joint: type fixed, parent panda_link2, child panda_link2_sc, origin rpy=0 0 0
- added joint panda_link3_sc_joint: type fixed, parent panda_link3, child panda_link3_sc, origin rpy=0 0 0
- added joint panda_link4_sc_joint: type fixed, parent panda_link4, child panda_link4_sc, origin rpy=0 0 0
- added joint panda_link5_sc_joint: type fixed, parent panda_link5, child panda_link5_sc, origin rpy=0 0 0
- added joint panda_link6_sc_joint: type fixed, parent panda_link6, child panda_link6_sc, origin rpy=0 0 0
- added joint panda_link7_sc_joint: type fixed, parent panda_link7, child panda_link7_sc, origin rpy=0 0 0.7853981633974483
- added joint panda_tcp_ball_joint: type fixed, parent panda_hand_tcp, child panda_ball, origin xyz=-4.985383226574662e-05 -0.00013336514178627587 0.028808917565181256 rpy=0.0 0.0 0.0
- joint panda_finger_joint1: axis (none) -> 0 1 0; limit (none) -> lower=0.0 upper=0.04 effort=100 velocity=0.2; type fixed -> prismatic
- joint panda_finger_joint2: axis (none) -> 0 -1 0; limit (none) -> lower=0.0 upper=0.04 effort=100 velocity=0.2; mimic (none) -> joint=panda_finger_joint1; type fixed -> prismatic
- joint panda_joint1: origin xyz=0 0 0.333 rpy=0 0 0 -> xyz=1.0781376906493187e-16 -1.8834554812913657e-16 0.3330000000000003 rpy=-0.003983554629324744 -3.0445592280821456e-06 -1.415091495734401e-16
- joint panda_joint2: origin xyz=0 0 0 rpy=-1.5707963267948966 0 0 -> xyz=0.00016341912877901506 -0.00017156737387569485 5.375629426571536e-16 rpy=-1.5727904750994823 0.0012540685707349425 1.1013797442415149e-06
- joint panda_joint3: origin xyz=0 -0.316 0 rpy=1.5707963267948966 0 0 -> xyz=0.0001299051404350041 -0.3135816347471088 -0.00017155993521596554 rpy=1.572162461367731 0.0006574297825724241 0.001194814825299022
- joint panda_joint4: origin xyz=0.0825 0 0 rpy=1.5707963267948966 0 0 -> xyz=0.08146886587596877 7.5485817626186065e-06 -0.0024217097938806077 rpy=1.5730691786583635 0.012312431691333916 -0.0006583382654092967
- joint panda_joint5: origin xyz=-0.0825 0.384 0 rpy=-1.5707963267948966 0 0 -> xyz=-0.07777374924834445 0.3814887482917348 5.983080398729339e-06 rpy=-1.5699403519499557 0.005136687763343844 -0.01071152681808784
- joint panda_joint6: origin xyz=0 0 0 rpy=1.5707963267948966 0 0 -> xyz=0.000550003505381384 2.4422161132276864e-05 -0.002451620682018998 rpy=1.5705975004428918 -0.0003904054404951994 0.005129001217567927
- joint panda_joint7: origin xyz=0.088 0 0 rpy=1.5707963267948966 0 0 -> xyz=0.08896699606060197 0.0011974566380215954 -2.2321885163227118e-05 rpy=1.570874805280769 -8.16444341763457e-07 0.00028739172352703387
